File: TSSOP16_Breakout_Boards/TSSOP_16_Breakout_Board.kicad_pcb (KiCad board)
At the start: 2 copper layers, 26.5 x 25 mm, 6 parts, among them J1 Conn_01x08, J2 Conn_01x08, J3 Conn_01x01, J4 Conn_01x01

Commit message: finalized tssop 16 board
Parts:
- removed SOIC16: 16_Pin_SOIC_Board, SOIC_Footprints:16_Pin_SOIC_Board
- added TSSOP16: 16_Pin_TSSOP_Board, TSSOP_Footprints:16_Pin_TSSOP_Board, F.Cu at (158.9, 100.6)
Routing:
- net Net-(J1-Pad8): track 9.86 -> 11.6 mm
- net Net-(J2-Pad1): track 9.86 -> 11.6 mm
- net Net-(J2-Pad8): track 9.86 -> 11.6 mm
- net Net-(J1-Pad1): track 9.86 -> 11.6 mm
- net Net-(J1-Pad7): track 8.45 -> 9.78 mm
- net Net-(J2-Pad7): track 8.45 -> 9.78 mm
- net Net-(J2-Pad2): track 8.45 -> 9.78 mm
- net Net-(J1-Pad2): track 8.45 -> 9.78 mm
- net Net-(J2-Pad6): track 7.05 -> 7.95 mm
- net Net-(J1-Pad6): track 7.05 -> 7.95 mm
- net Net-(J1-Pad3): track 7.05 -> 7.95 mm
- net Net-(J2-Pad3): track 7.05 -> 7.95 mm
Other:
- board text added: "16 Pin TSSOP Breakout Board"
- board text removed: "16 Pin SOIC Breakout Board"
