File: TSSOP16_Breakout_Boards/TSSOP_16_Breakout_Board.kicad_sch (KiCad schematic)
At the start: 6 parts, among them J1 Conn_01x08, J2 Conn_01x08, J3 Conn_01x01, J4 Conn_01x01

Commit message: finalized tssop 16 board
Parts:
- TSSOP1: footprint (none) -> TSSOP_Footprints:16_Pin_TSSOP_Board
Changed lines of the file:
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@@
     (property "Reference" "TSSOP1" (id 0) (at 138.43 109.22 0))
     (property "Value" "16_Pin_TSSOP_Board" (id 1) (at 138.43 111.76 0))
-    (property "Footprint" "" (id 2) (at 138.43 97.79 0)
+    (property "Footprint" "TSSOP_Footprints:16_Pin_TSSOP_Board" (id 2) (at 138.43 97.79 0)
       (effects (font (size 1.27 1.27)) hide)
     )
@@
     )
     (path "/f5ada240-c394-4ad1-b253-0f8c493bffaf"
-      (reference "TSSOP1") (unit 1) (value "16_Pin_TSSOP_Board") (footprint "")
+      (reference "TSSOP1") (unit 1) (value "16_Pin_TSSOP_Board") (footprint "TSSOP_Footprints:16_Pin_TSSOP_Board")
     )
   )
