File: TSSOP20_Breakout_Boards/TSSOP_20_Breakout_Board.kicad_sch (KiCad schematic)
At the start: 6 parts, among them J1 Conn_01x10, J2 Conn_01x10, J3 Conn_01x01, J4 Conn_01x01

Commit message: finalized tssop 20 design
Parts:
- TSSOP1: footprint (none) -> TSSOP_Footprints:20_Pin_TSSOP_Board
Changed lines of the file:
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@@
     (property "Reference" "TSSOP1" (id 0) (at 125.73 120.65 0))
     (property "Value" "20_Pin_TSSOP_Board" (id 1) (at 125.73 123.19 0))
-    (property "Footprint" "" (id 2) (at 127 107.95 0)
+    (property "Footprint" "TSSOP_Footprints:20_Pin_TSSOP_Board" (id 2) (at 127 107.95 0)
       (effects (font (size 1.27 1.27)) hide)
     )
@@
     )
     (path "/04466a57-d90b-41a1-86f7-0a72597bfeae"
-      (reference "TSSOP1") (unit 1) (value "20_Pin_TSSOP_Board") (footprint "")
+      (reference "TSSOP1") (unit 1) (value "20_Pin_TSSOP_Board") (footprint "TSSOP_Footprints:20_Pin_TSSOP_Board")
     )
   )
